Commit message: finish debugging Jacobian.py. It seems to have singularity within.

File: project/proj2_baseball/rsc/robotarm/urdf/robotarm1.urdf (robot description, URDF)
Before this commit: robot robotarm, 10 links, 9 joints
Links:
- removed link catcher_lower
- removed link catcher_upper
- removed link link1
- removed link link2
- removed link link3
- removed link link4
- removed link link5
- removed link link6
- removed link link7
- removed link link8
- added link Catcher_Lower, mass 0.087826; collision mesh filename=package://robotarm1/meshes/Catcher_Lower.STL; visual mesh filename=package://robotarm1/meshes/Catcher_Lower.STL
- added link Catcher_Upper, mass 0.13937; collision mesh filename=package://robotarm1/meshes/Catcher_Upper.STL; visual mesh filename=package://robotarm1/meshes/Catcher_Upper.STL
- added link Link_1, mass 0.968515917956123; collision mesh filename=package://robotarm1/meshes/Link_1.STL; visual mesh filename=package://robotarm1/meshes/Link_1.STL
- added link Link_2, mass 1.28853409511538; collision mesh filename=package://robotarm1/meshes/Link_2.STL; visual mesh filename=package://robotarm1/meshes/Link_2.STL
- added link Link_3, mass 1.18174149257434; collision mesh filename=package://robotarm1/meshes/Link_3.STL; visual mesh filename=package://robotarm1/meshes/Link_3.STL
- added link Link_4, mass 1.28909961850142; collision mesh filename=package://robotarm1/meshes/Link_4.STL; visual mesh filename=package://robotarm1/meshes/Link_4.STL
- added link Link_5, mass 1.20648390273837; collision mesh filename=package://robotarm1/meshes/Link_5.STL; visual mesh filename=package://robotarm1/meshes/Link_5.STL
- added link Link_6, mass 0.86991; collision mesh filename=package://robotarm1/meshes/Link_6.STL; visual mesh filename=package://robotarm1/meshes/Link_6.STL
- added link Link_7, mass 0.509047523656065; collision mesh filename=package://robotarm1/meshes/Link_7.STL; visual mesh filename=package://robotarm1/meshes/Link_7.STL
- added link base_link, mass 5.6925658883047; collision mesh filename=package://robotarm1/meshes/base_link.STL; visual mesh filename=package://robotarm1/meshes/base_link.STL
Joints:
- removed joint joint1to2
- removed joint joint2to3
- removed joint joint3to4
- removed joint joint4to5
- removed joint joint5to6
- removed joint joint6to7
- removed joint joint7to8
- removed joint joint_lower
- removed joint joint_upper
- added joint Catcher_Joint_Lower: type continuous, parent Link_7, child Catcher_Lower, origin xyz=0.0600000000000073 -0.00750000000000006 0 rpy=1.57079632679492 0 0, axis 0 1 0
- added joint Catcher_Joint_Upper: type continuous, parent Link_7, child Catcher_Upper, origin xyz=0.0600000000000074 0.00750000000000006 0 rpy=-1.57079632679487 0 0, axis 0 1 0
- added joint Joint_1: type continuous, parent base_link, child Link_1, origin xyz=0 0 0.1652 rpy=1.5708 0 0, axis 0 1 0
- added joint Joint_2: type continuous, parent Link_1, child Link_2, origin xyz=0.112400000000005 0.0500000000000001 0 rpy=0 0 0, axis 1 0 0
- added joint Joint_3: type continuous, parent Link_2, child Link_3, origin xyz=0 0.351 0 rpy=0 0 0, axis 1 0 0
- added joint Joint_4: type continuous, parent Link_3, child Link_4, origin xyz=-0.0624 0 0 rpy=0 0 0, axis 1 0 0
- added joint Joint_5: type continuous, parent Link_4, child Link_5, origin xyz=0 0.3512 0 rpy=0 0 0, axis 1 0 0
- added joint Joint_6: type continuous, parent Link_5, child Link_6, origin xyz=0.1124 0 0 rpy=0 0 0, axis 0 1 0
- added joint Joint_7: type continuous, parent Link_6, child Link_7, origin xyz=0 0.1124 0 rpy=0 0 0, axis 1 0 0
