Commit message: solve the bug for not being able to rotate

File: project/proj2_baseball/rsc/robotarm/urdf/robotarm.urdf (robot description, URDF)
Before this commit: robot robotarm, 10 links, 9 joints
Joints:
- joint joint1to2: limit lower=0 upper=0 effort=0 velocity=0 -> (none)
- joint joint2to3: limit lower=0 upper=0 effort=0 velocity=0 -> (none)
- joint joint3to4: limit lower=0 upper=0 effort=0 velocity=0 -> (none)
- joint joint4to5: limit lower=0 upper=0 effort=0 velocity=0 -> (none)
- joint joint5to6: limit lower=0 upper=0 effort=0 velocity=0 -> (none)
- joint joint6to7: limit lower=0 upper=0 effort=0 velocity=0 -> (none)
- joint joint_lower: limit lower=0 upper=0 effort=0 velocity=0 -> (none)
- joint joint_upper: limit lower=0 upper=0 effort=0 velocity=0 -> (none)

Commit message: modified urdf origin axis

File: project/proj2_baseball/rsc/robotarm/urdf/robotarm.urdf (robot description, URDF)
Before this commit: robot robotarm, 10 links, 9 joints
Links:
- link catcher_lower: mass 0.0344733076025474 -> 0.034473
- link catcher_upper: mass 0.0721393119023469 -> 0.072139
- link link1: mass 0 -> 5.6926
- link link2: mass 0.968515917956123 -> 0.96852
- link link3: mass 1.28853409511538 -> 1.2885
- link link4: mass 1.18174149257434 -> 1.1817
- link link5: mass 1.28909961850142 -> 1.2891
- link link6: mass 1.20648390273837 -> 1.2065
- link link7: mass 0.869909136744433 -> 0.86991
- link link8: mass 0.509047523656065 -> 0.50905
Joints:
- joint joint3to4: origin xyz=0 0.351 0 rpy=0.79634 0 0 -> xyz=0 0.351 0 rpy=0 0 0
- joint joint4to5: axis 1 0 0 -> 0 0 0; origin xyz=-0.1624 0.2456 -0.25104 rpy=-0.79634 0 0 -> xyz=-0.1624 0.3512 0 rpy=0 0 0
- joint joint_lower: origin xyz=0.0600000000000061 -0.00750000000000006 0 rpy=1.5707963267949 0 -0.602113242360167 -> xyz=0.06 -0.0075 0 rpy=1.5708 0 -0.60211

Commit message: catcher orientation modified

File: project/proj2_baseball/rsc/robotarm/urdf/robotarm.urdf (robot description, URDF)
Before this commit: robot robotarm, 10 links, 9 joints
Links:
- link catcher_lower: mass 0.034473 -> 0.0344733076025474
- link catcher_upper: mass 0.072139 -> 0.0721393119023468
- link link1: mass 5.6926 -> 5.6925658883047
- link link2: mass 0.96852 -> 0.968515917956123
- link link3: mass 1.2885 -> 1.28853409511538
- link link4: mass 1.1817 -> 1.18174149257434
- link link5: mass 1.2891 -> 1.28909961850142
- link link6: mass 1.2065 -> 1.20648390273837
- link link7: mass 0.86991 -> 0.869909136744433
- link link8: mass 0.50905 -> 0.509047523656065
Joints:
- joint joint1to2: origin xyz=0 0 0.2152 rpy=1.5708 0 0 -> xyz=0 0 0.2152 rpy=1.5707963267949 0 0
- joint joint5to6: origin xyz=0.1624 0 0 rpy=0 0 0 -> xyz=0.162399999999994 0 0 rpy=0 0 0
- joint joint6to7: origin xyz=0 0.1124 0 rpy=0 0 0 -> xyz=0 0.112399999999999 0 rpy=0 0 0
- joint joint_lower: origin xyz=0.06 -0.0075 0 rpy=1.5708 0 -0.60211 -> xyz=0.0600000000000061 -0.00750000000000006 0 rpy=1.5707963267949 0 0
- joint joint_upper: origin xyz=0.06 0.0075 0 rpy=-1.5708 0 0.58786 -> xyz=0.05 0 0 rpy=-1.5707963267949 0 0

Commit message: modify the model of catcher debugging Jacobian.py

File: project/proj2_baseball/rsc/robotarm/urdf/robotarm.urdf (robot description, URDF)
Before this commit: robot robotarm, 10 links, 9 joints
Links:
- link catcher_lower: mass 0.0344733076025474 -> 0.0720761747561821
- link catcher_upper: mass 0.0721393119023468 -> 0.11687084901057

Commit message: modify the model, design the path of the tip of the robot arm, concave problem remains to be solved

File: project/proj2_baseball/rsc/robotarm/urdf/robotarm.urdf (robot description, URDF)
Before this commit: robot robotarm, 10 links, 9 joints
Links:
- removed link catcher_lower
- removed link catcher_upper
- removed link link1
- removed link link2
- removed link link3
- removed link link4
- removed link link5
- removed link link6
- removed link link7
- removed link link8
- added link Catcher_Lower, mass 0.257146155727528; collision mesh filename=package://robotarm/meshes/Catcher_Lower.STL; visual mesh filename=package://robotarm/meshes/Catcher_Lower.STL
- added link Catcher_Upper, mass 0.265488660995906; collision mesh filename=package://robotarm/meshes/Catcher_Upper.STL; visual mesh filename=package://robotarm/meshes/Catcher_Upper.STL
- added link Link_1, mass 0.968515917956123; collision mesh filename=package://robotarm/meshes/Link_1.STL; visual mesh filename=package://robotarm/meshes/Link_1.STL
- added link Link_2, mass 1.28853409511538; collision mesh filename=package://robotarm/meshes/Link_2.STL; visual mesh filename=package://robotarm/meshes/Link_2.STL
- added link Link_3, mass 1.18174149257434; collision mesh filename=package://robotarm/meshes/Link_3.STL; visual mesh filename=package://robotarm/meshes/Link_3.STL
- added link Link_4, mass 1.28909961850142; collision mesh filename=package://robotarm/meshes/Link_4.STL; visual mesh filename=package://robotarm/meshes/Link_4.STL
- added link Link_5, mass 1.20648390273837; collision mesh filename=package://robotarm/meshes/Link_5.STL; visual mesh filename=package://robotarm/meshes/Link_5.STL
- added link Link_6, mass 0.869909136744433; collision mesh filename=package://robotarm/meshes/Link_6.STL; visual mesh filename=package://robotarm/meshes/Link_6.STL
- added link Link_7, mass 0.509047523656065; collision mesh filename=package://robotarm/meshes/Link_7.STL; visual mesh filename=package://robotarm/meshes/Link_7.STL
- added link base_link, mass 5.6925658883047; collision mesh filename=package://robotarm/meshes/base_link.STL; visual mesh filename=package://robotarm/meshes/base_link.STL
Joints:
- removed joint joint1to2
- removed joint joint2to3
- removed joint joint3to4
- removed joint joint4to5
- removed joint joint5to6
- removed joint joint6to7
- removed joint joint7to8
- removed joint joint_lower
- removed joint joint_upper
- added joint Catcher_Joint_Lower: type continuous, parent Link_7, child Catcher_Lower, origin xyz=0.0600000000000073 -0.00750000000000006 0 rpy=1.57079632679492 0 0, axis 0 1 0
- added joint Catcher_Joint_Upper: type continuous, parent Link_7, child Catcher_Upper, origin xyz=0.0600000000000074 0.00750000000000006 0 rpy=-1.57079632679487 0 0, axis 0 1 0
- added joint Joint_1: type continuous, parent base_link, child Link_1, origin xyz=0 0 0.1652 rpy=1.5707963267949 0 0, axis 0 1 0
- added joint Joint_2: type continuous, parent Link_1, child Link_2, origin xyz=0.112400000000005 0.0500000000000001 0 rpy=0 0 0, axis 1 0 0
- added joint Joint_3: type continuous, parent Link_2, child Link_3, origin xyz=0 0.351 0 rpy=0 0 0, axis 1 0 0
- added joint Joint_4: type continuous, parent Link_3, child Link_4, origin xyz=-0.0624000000000001 0 0 rpy=0 0 0, axis 1 0 0
- added joint Joint_5: type continuous, parent Link_4, child Link_5, origin xyz=0 0.3512 0 rpy=0 0 0, axis 1 0 0
- added joint Joint_6: type continuous, parent Link_5, child Link_6, origin xyz=0.112399999999994 0 0 rpy=0 0 0, axis 0 1 0
- added joint Joint_7: type continuous, parent Link_6, child Link_7, origin xyz=0 0.112399999999999 0 rpy=0 0 0, axis 1 0 0

Commit message: catcher modified

File: project/proj2_baseball/rsc/robotarm/urdf/robotarm.urdf (robot description, URDF)
Before this commit: robot robotarm, 10 links, 9 joints
Links:
- link Catcher_Lower: mass 0.257146155727528 -> 0.316579012529707
- link Catcher_Upper: mass 0.265488660995906 -> 0.324921517798083
Joints:
- joint Joint_4: origin xyz=-0.0624000000000001 0 0 rpy=0 0 0 -> xyz=-0.0624 0 0 rpy=0 0 0
- joint Joint_6: origin xyz=0.112399999999994 0 0 rpy=0 0 0 -> xyz=0.1124 0 0 rpy=0 0 0

Commit message: model modified

File: project/proj2_baseball/rsc/robotarm/urdf/robotarm.urdf (robot description, URDF)
Before this commit: robot robotarm, 10 links, 9 joints
Links:
- link Catcher_Lower: mass 0.316579012529707 -> 0.408159928023487
- link Catcher_Upper: mass 0.324921517798083 -> 0.416502433291861
- link Link_7: mass 0.509047523656065 -> 0.509050484778038
Joints:
- joint Joint_4: origin xyz=-0.0624 0 0 rpy=0 0 0 -> xyz=-0.0624000000000001 0 0 rpy=0 0 0
- joint Joint_6: origin xyz=0.1124 0 0 rpy=0 0 0 -> xyz=0.112399999999994 0 0 rpy=0 0 0
