Commit message: fy test passed

File: project/proj4_run/rsc/MarioTheRobot.urdf (robot description, URDF)
Before this commit: robot Mario, 7 links, 6 joints
Joints:
- joint World2XAxis: type prismatic -> fixed
- joint XAxis2ZAxis: type prismatic -> fixed
- joint ZAxis2body: type continuous -> fixed

Commit message: theta test passed

File: project/proj4_run/rsc/MarioTheRobot.urdf (robot description, URDF)
Before this commit: robot Mario, 7 links, 6 joints
Joints:
- joint ZAxis2body: type fixed -> continuous
- joint engine1: type continuous -> fixed

Commit message: x test passed

File: project/proj4_run/rsc/MarioTheRobot.urdf (robot description, URDF)
Before this commit: robot Mario, 7 links, 6 joints
Joints:
- joint engine1: type fixed -> continuous

Commit message: v_theta, v_fy, v_x test passed

File: project/proj4_run/rsc/MarioTheRobot.urdf (robot description, URDF)
Before this commit: robot Mario, 7 links, 6 joints
Joints:
- joint ZAxis2body: type continuous -> fixed

Commit message: Dev v1.0

File: project/proj4_run/rsc/MarioTheRobot.urdf (robot description, URDF)
Before this commit: robot Mario, 7 links, 6 joints
Links:
- link body: mass 5.0 -> 7.0
- link leg: mass 0.5 -> 0.05
- link thigh: mass 0.5 -> 0.05
- link wheel: mass 1.0 -> 2.0
